File: hardware/prototype_5kW/variable_frequency_drive.kicad_sch (KiCad schematic)
At the start: 110 parts, among them J1 KSE-25C-B-03P, J2 SWD, J3 KSE-25C-B-02P, K1 HJQ-15F-12VDC-S-Z, Q1 2SC1384, SW9 RotaryEncoder_Switch, U1 STM32F401CCUx, U2 FSAM50SM60A, U3 LM358, U4 ACS758-050B, U5 ACS758-050B, U6 TM1637, U7 CC56-12GWA, U8 LD1117S33TR, Y1 25MHz

Commit message: Changed the structure of the project
Parts:
- removed FL1: Filter_EMI_LL, symbol Device:Filter_EMI_LL
- added C?: 4.7uF, symbol Device:C
- added C?: 470uF, symbol Device:C
- added C? (x2): 22pF, symbol Device:C
- added C?: 1nF, symbol Device:C
- added C?: 100nF, symbol Device:C
- added C?: 220pF, symbol Device:C
- added R?: 10k, symbol Device:R
- added R?: 1k, symbol Device:R
- added U?: STM32F401RBTx, Package_QFP:LQFP-64_10x10mm_P0.5mm, symbol MCU_ST_STM32F4:STM32F401RBTx
- added Y?: 25MHz, symbol Device:Crystal
- R?: Power (none) -> 5W
Connections:
- net +3.3V: now also R?.1
- net CLK: now also U?.61 (PB8)
- net DIO: now also U?.62 (PB9)
- net ENCODER_S1: now also U?.50 (PA15)
- net ENCODER_S2: now also U?.55 (PB3)
- net FAULT: now also U?.33 (PB12)
- net GND: now also C?.1, C?.1, C?.1, C?.1, C?.1, C?.2, C?.2, R?.1, U?.12 (VSSA), U?.18 (VSS), U?.31 (VSS), U?.47 (VSS), U?.63 (VSS)
- net L: now also D5.4
- net N: now also D5.2
- net NTC_BP: now also U?.29 (PB10)
- net UH: now also U?.34 (PB13)
- net UL: now also U?.41 (PA8)
- net VH: now also U?.35 (PB14)
- net VL: now also U?.42 (PA9)
- net WH: now also U?.36 (PB15)
- net WL: now also U?.43 (PA10)
- new net: C?.1, U?.30 (VCAP1)
- new net: C?.2, C?.2, C?.2, U?.19 (VDD), U?.32 (VDD), U?.48 (VDD), U?.64 (VDD)
- new net: C?.2, U?.6 (PH1), Y?.2
- new net: R?.2, U?.60 (BOOT0)
- new net: C?.2, U?.5 (PH0), Y?.1
- new net: C?.1, R?.2, U?.7 (NRST)
- no-connect marks 17 -> 18
Other:
- moved on the sheet: C21, C22, C26, C27, C28, C29, C30, C31, C32, C33, C7, D4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
